File: Hardware/InkTime.brd (EAGLE design)
At the start: 46 x 35 mm, 105 parts, among them IC1 BQ25180YBGR, IC2 DRV2605YZFR, IC3 BMA421, IC9 RT6160AWSC, J1 503480-2400, J2 TC2030-IDC, J4 KH-TYPE-C-16P, Q1 20V/4.2A/52mΩ/1.4W, Q3 SI1308EDL-T1-GE3, U1 NRF52840_QF, U3 MAX17048G+T10, X1 32MHz, X2 32.768kHz

Commit message: Updated Hardware
Parts:
- SW_DN, SW_ENT, SW_UP: value 2025-10-22_07-23-44_LIBRARY_EVP-AKE31ASW_EVP-AKE31A_PAN -> 2025-10-22_07-23-44_LIBRARY_EVP-AKE31A
- moved C25 204.9 mm to (-6.20, 3.20), turned to 90 degrees
- moved C24 184.5 mm to (-6.70, 8.50), turned to 270 degrees
- moved C33 179.6 mm to (-5.20, 3.20), turned to 90 degrees
- moved R2 163.4 mm to (-7.80, 4.90), turned to 90 degrees
- moved R4 161.4 mm to (-7.80, 5.50), turned to 90 degrees
- moved IC9 157.3 mm to (-6.20, 5.90)
- moved C23 151.8 mm to (-5.80, 8.30), turned to 270 degrees
- moved TP_VREG 149.5 mm to (-2.60, 3.30)
- moved TP_3V3 146.1 mm to (-9.50, 8.90)
- moved X1 137.2 mm to (16.6, 10.1), turned to 90 degrees
- moved U3 133.2 mm to (-17.6, 10.5), turned to 270 degrees
- moved X2 128.5 mm to (5.50, 7.40), turned to 270 degrees
- moved TP_VBAT 122.5 mm to (-18.7, 13.4), turned to 270 degrees
- moved TP_3.3V 101.4 mm to (8.50, 15.1)
- moved TP_BAT_GND 101.1 mm to (-20.2, 11.4), turned to 270 degrees
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Connections:
- net 3V1 renamed CACA2
Routing:
- net VBAT: track 0.00 -> 314.2 mm, vias 0 -> 6
- net 3V3: track 0.00 -> 157.7 mm, vias 0 -> 18
- net SCL: track 0.00 -> 102.1 mm, vias 0 -> 12
- net SDA: track 0.00 -> 101.5 mm, vias 0 -> 11
- net GND: track 0.00 -> 79.7 mm, vias 0 -> 65
- net MOSI: track 0.00 -> 69.4 mm, vias 0 -> 6
- net EPD_RST: track 0.00 -> 48.4 mm, vias 0 -> 2
- net ALERT: track 0.00 -> 46.8 mm, vias 0 -> 8
- net EPD_BUSY: track 0.00 -> 46.6 mm, vias 0 -> 6
- net VBUS: track 0.00 -> 46.0 mm, vias 0 -> 3
- net SCK: track 0.00 -> 45.6 mm, vias 0 -> 4
- net EPD_3V3: track 0.00 -> 41.6 mm, vias 0 -> 4
- net HAPTIC_EN: track 0.00 -> 36.7 mm, vias 0 -> 6
- net EPD_DC: track 0.00 -> 34.7 mm, vias 0 -> 6
- net P0.13: track 0.00 -> 34.3 mm, vias 0 -> 2
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