File: Hardware/Schematic.sch (EAGLE design)
At the start: 105 parts, among them IC1 BQ25180YBGR, IC2 DRV2605YZFR, IC3 BMA421, IC9 RT6160AWSC, J1 503480-2400, J2 TC2030-IDC, J4 KH-TYPE-C-16P, Q1 20V/4.2A/52mΩ/1.4W, Q3 SI1308EDL-T1-GE3, U1 NRF52840_QF, U3 MAX17048G+T10, X1 32MHz, X2 32.768kHz

Commit message: Updated Hardware
Parts:
- SW_DN, SW_ENT, SW_UP: value 2025-10-22_07-23-44_LIBRARY_EVP-AKE31ASW_EVP-AKE31A_PAN -> 2025-10-22_07-23-44_LIBRARY_EVP-AKE31A; device InkTime_v5:2025-10-22_07-23-44_LIBRARY_EVP-AKE31ASW_EVP-AKE31A_PAN -> InkTime_v5:2025-10-22_07-23-44_LIBRARY_EVP-AKE31A
Connections:
- net 3V1 renamed CACA2
